File: cpu.sch (KiCad schematic (older format))
At the start: 23 parts, among them IC20 74LS373, IC21 74LS245, IC22 74LS373, IC23 8088_Max_Mode, IC24 8087, IC29 74LS27, IC30 74LS244_Split, IC39 74LS245, IC40 8288, IC52 74LS04, IC67 74LS20, IC68 74LS10, IC69 74LS74, IC70 74S00, IC83 74LS32, IC84 74LS00, IC85 74LS04, IC86 74LS74, IC87 74LS175, IC88 74LS08

Commit message: Tidy up and map all signals
This fixes up the schematic to:
 - Look presentable
 - Fix all labels connecting sheets
 - Tidy up all loose ends by either inspecting the PCB under
    magnification, measuring with an oscillosope or buzzing
    out with a meter
 - Pass ERC (with 1 exception due to incorrect circuitry around
    pin 33 on the FPU (~RQ~/~GT1~)
Parts:
- removed IC29: 74LS27, symbol 74xx:74LS27
- removed IC67: 74LS20, symbol 74xx:74LS20
- removed IC68: 74LS10, symbol 74xx:74LS10
- removed IC69, IC86: 74LS74, symbol 74xx:74LS74
- removed IC70: 74S00, symbol 74xx:74LS00
- removed IC83: 74LS32, symbol 74xx:74LS32
- removed IC84: 74LS00, symbol 74xx:74LS00
- removed IC85: 74LS04, symbol 74xx:74LS04
- removed IC87: 74LS175, symbol 74xx:74LS175
- removed IC88: 74LS08, symbol 74xx:74LS08
- removed R17: 4K7, symbol Device:R
- removed RP5: 4K7, Resistor_THT:R_Array_SIP9, symbol Device:R_Network08
- added RP5: 4K7, Resistor_THT:R_Array_SIP9, symbol Device:R_Network08_Split
- IC23: value 8088_Max_Mode -> 8088-2
- renumbered RP3 to RP2
Connections:
- net +5V: now also IC20.20 (VCC), IC21.20 (VCC), IC22.20 (VCC), IC23.40 (VCC), IC24.40 (VCC), IC39.20 (VCC), IC40.20 (VCC), RP5.1 (R1.1)
- net GND: now also IC21.10 (GND), IC22.10 (GND)
- net ~RQ~-~GT0~: now also RP5.2 (R1.2)
- net ~TEST~: now also RP5.8 (R7.2)
- net INT: now reaches IC23.18 (INTR)
- net ~DATA_EN~: now reaches IC21.19 (CE), IC52.8
- removed net XXX: IC39.6 (A4), IC39.7 (A5), IC39.8 (A6), IC39.9 (A7), IC40.11 (~IOWC~), IC40.9 (~MWTC~)
- no-connect marks 3 -> 13
Other:
- moved on the sheet: IC20, IC21, IC22, IC30A, IC39, IC40, IC52D, RP2
