File: ram.sch (KiCad schematic (older format))
At the start: 0 parts

Commit message: Tidy up and map all signals
This fixes up the schematic to:
 - Look presentable
 - Fix all labels connecting sheets
 - Tidy up all loose ends by either inspecting the PCB under
    magnification, measuring with an oscillosope or buzzing
    out with a meter
 - Pass ERC (with 1 exception due to incorrect circuitry around
    pin 33 on the FPU (~RQ~/~GT1~)
Parts:
- added IC43, IC44, IC45, IC46, IC47, IC48, IC49, IC50, IC51, IC57, IC58, IC59, IC60, IC61, IC62, IC63, IC64, IC65, IC72, IC73, IC74, IC75, IC76, IC77, IC78, IC79, IC80, IC89, IC90, IC91, IC92, IC93, IC94, IC95, IC96, IC97: TMS4256, symbol PCII-System-Board-Custom-Parts:TMS4256
Connections:
- new net +5V: IC43.8 (VDD), IC44.8 (VDD), IC45.8 (VDD), IC46.8 (VDD), IC47.8 (VDD), IC48.8 (VDD), IC49.8 (VDD), IC50.8 (VDD), IC51.8 (VDD), IC57.8 (VDD), IC58.8 (VDD), IC59.8 (VDD), IC60.8 (VDD), IC61.8 (VDD), IC62.8 (VDD), IC63.8 (VDD), IC64.8 (VDD), IC65.8 (VDD), IC72.8 (VDD), IC73.8 (VDD), IC74.8 (VDD), IC75.8 (VDD), IC76.8 (VDD), IC77.8 (VDD), IC78.8 (VDD), IC79.8 (VDD), IC80.8 (VDD), IC89.8 (VDD), IC90.8 (VDD), IC91.8 (VDD), IC92.8 (VDD), IC93.8 (VDD), IC94.8 (VDD), IC95.8 (VDD), IC96.8 (VDD), IC97.8 (VDD)
- new net GND: IC43.16 (VSS), IC44.16 (VSS), IC45.16 (VSS), IC46.16 (VSS), IC47.16 (VSS), IC48.16 (VSS), IC49.16 (VSS), IC50.16 (VSS), IC51.16 (VSS), IC57.16 (VSS), IC58.16 (VSS), IC59.16 (VSS), IC60.16 (VSS), IC61.16 (VSS), IC62.16 (VSS), IC63.16 (VSS), IC64.16 (VSS), IC65.16 (VSS), IC72.16 (VSS), IC73.16 (VSS), IC74.16 (VSS), IC75.16 (VSS), IC76.16 (VSS), IC77.16 (VSS), IC78.16 (VSS), IC79.16 (VSS), IC80.16 (VSS), IC89.16 (VSS), IC90.16 (VSS), IC91.16 (VSS), IC92.16 (VSS), IC93.16 (VSS), IC94.16 (VSS), IC95.16 (VSS), IC96.16 (VSS), IC97.16 (VSS)
- new net MA0: IC43.5 (A0), IC44.5 (A0), IC45.5 (A0), IC46.5 (A0), IC47.5 (A0), IC48.5 (A0), IC49.5 (A0), IC50.5 (A0), IC51.5 (A0), IC57.5 (A0), IC58.5 (A0), IC59.5 (A0), IC60.5 (A0), IC61.5 (A0), IC62.5 (A0), IC63.5 (A0), IC64.5 (A0), IC65.5 (A0), IC72.5 (A0), IC73.5 (A0), IC74.5 (A0), IC75.5 (A0), IC76.5 (A0), IC77.5 (A0), IC78.5 (A0), IC79.5 (A0), IC80.5 (A0), IC89.5 (A0), IC90.5 (A0), IC91.5 (A0), IC92.5 (A0), IC93.5 (A0), IC94.5 (A0), IC95.5 (A0), IC96.5 (A0), IC97.5 (A0)
- new net MA1: IC43.7 (A1), IC44.7 (A1), IC45.7 (A1), IC46.7 (A1), IC47.7 (A1), IC48.7 (A1), IC49.7 (A1), IC50.7 (A1), IC51.7 (A1), IC57.7 (A1), IC58.7 (A1), IC59.7 (A1), IC60.7 (A1), IC61.7 (A1), IC62.7 (A1), IC63.7 (A1), IC64.7 (A1), IC65.7 (A1), IC72.7 (A1), IC73.7 (A1), IC74.7 (A1), IC75.7 (A1), IC76.7 (A1), IC77.7 (A1), IC78.7 (A1), IC79.7 (A1), IC80.7 (A1), IC89.7 (A1), IC90.7 (A1), IC91.7 (A1), IC92.7 (A1), IC93.7 (A1), IC94.7 (A1), IC95.7 (A1), IC96.7 (A1), IC97.7 (A1)
- new net MA2: IC43.6 (A2), IC44.6 (A2), IC45.6 (A2), IC46.6 (A2), IC47.6 (A2), IC48.6 (A2), IC49.6 (A2), IC50.6 (A2), IC51.6 (A2), IC57.6 (A2), IC58.6 (A2), IC59.6 (A2), IC60.6 (A2), IC61.6 (A2), IC62.6 (A2), IC63.6 (A2), IC64.6 (A2), IC65.6 (A2), IC72.6 (A2), IC73.6 (A2), IC74.6 (A2), IC75.6 (A2), IC76.6 (A2), IC77.6 (A2), IC78.6 (A2), IC79.6 (A2), IC80.6 (A2), IC89.6 (A2), IC90.6 (A2), IC91.6 (A2), IC92.6 (A2), IC93.6 (A2), IC94.6 (A2), IC95.6 (A2), IC96.6 (A2), IC97.6 (A2)
- new net MA3: IC43.12 (A3), IC44.12 (A3), IC45.12 (A3), IC46.12 (A3), IC47.12 (A3), IC48.12 (A3), IC49.12 (A3), IC50.12 (A3), IC51.12 (A3), IC57.12 (A3), IC58.12 (A3), IC59.12 (A3), IC60.12 (A3), IC61.12 (A3), IC62.12 (A3), IC63.12 (A3), IC64.12 (A3), IC65.12 (A3), IC72.12 (A3), IC73.12 (A3), IC74.12 (A3), IC75.12 (A3), IC76.12 (A3), IC77.12 (A3), IC78.12 (A3), IC79.12 (A3), IC80.12 (A3), IC89.12 (A3), IC90.12 (A3), IC91.12 (A3), IC92.12 (A3), IC93.12 (A3), IC94.12 (A3), IC95.12 (A3), IC96.12 (A3), IC97.12 (A3)
- new net MA4: IC43.11 (A4), IC44.11 (A4), IC45.11 (A4), IC46.11 (A4), IC47.11 (A4), IC48.11 (A4), IC49.11 (A4), IC50.11 (A4), IC51.11 (A4), IC57.11 (A4), IC58.11 (A4), IC59.11 (A4), IC60.11 (A4), IC61.11 (A4), IC62.11 (A4), IC63.11 (A4), IC64.11 (A4), IC65.11 (A4), IC72.11 (A4), IC73.11 (A4), IC74.11 (A4), IC75.11 (A4), IC76.11 (A4), IC77.11 (A4), IC78.11 (A4), IC79.11 (A4), IC80.11 (A4), IC89.11 (A4), IC90.11 (A4), IC91.11 (A4), IC92.11 (A4), IC93.11 (A4), IC94.11 (A4), IC95.11 (A4), IC96.11 (A4), IC97.11 (A4)
- new net MA5: IC43.10 (A5), IC44.10 (A5), IC45.10 (A5), IC46.10 (A5), IC47.10 (A5), IC48.10 (A5), IC49.10 (A5), IC50.10 (A5), IC51.10 (A5), IC57.10 (A5), IC58.10 (A5), IC59.10 (A5), IC60.10 (A5), IC61.10 (A5), IC62.10 (A5), IC63.10 (A5), IC64.10 (A5), IC65.10 (A5), IC72.10 (A5), IC73.10 (A5), IC74.10 (A5), IC75.10 (A5), IC76.10 (A5), IC77.10 (A5), IC78.10 (A5), IC79.10 (A5), IC80.10 (A5), IC89.10 (A5), IC90.10 (A5), IC91.10 (A5), IC92.10 (A5), IC93.10 (A5), IC94.10 (A5), IC95.10 (A5), IC96.10 (A5), IC97.10 (A5)
- new net MA6: IC43.13 (A6), IC44.13 (A6), IC45.13 (A6), IC46.13 (A6), IC47.13 (A6), IC48.13 (A6), IC49.13 (A6), IC50.13 (A6), IC51.13 (A6), IC57.13 (A6), IC58.13 (A6), IC59.13 (A6), IC60.13 (A6), IC61.13 (A6), IC62.13 (A6), IC63.13 (A6), IC64.13 (A6), IC65.13 (A6), IC72.13 (A6), IC73.13 (A6), IC74.13 (A6), IC75.13 (A6), IC76.13 (A6), IC77.13 (A6), IC78.13 (A6), IC79.13 (A6), IC80.13 (A6), IC89.13 (A6), IC90.13 (A6), IC91.13 (A6), IC92.13 (A6), IC93.13 (A6), IC94.13 (A6), IC95.13 (A6), IC96.13 (A6), IC97.13 (A6)
- new net MA7: IC43.9 (A7), IC44.9 (A7), IC45.9 (A7), IC46.9 (A7), IC47.9 (A7), IC48.9 (A7), IC49.9 (A7), IC50.9 (A7), IC51.9 (A7), IC57.9 (A7), IC58.9 (A7), IC59.9 (A7), IC60.9 (A7), IC61.9 (A7), IC62.9 (A7), IC63.9 (A7), IC64.9 (A7), IC65.9 (A7), IC72.9 (A7), IC73.9 (A7), IC74.9 (A7), IC75.9 (A7), IC76.9 (A7), IC77.9 (A7), IC78.9 (A7), IC79.9 (A7), IC80.9 (A7), IC89.9 (A7), IC90.9 (A7), IC91.9 (A7), IC92.9 (A7), IC93.9 (A7), IC94.9 (A7), IC95.9 (A7), IC96.9 (A7), IC97.9 (A7)
- new net MA8: IC43.1 (A8), IC44.1 (A8), IC45.1 (A8), IC46.1 (A8), IC47.1 (A8), IC48.1 (A8), IC49.1 (A8), IC50.1 (A8), IC51.1 (A8), IC57.1 (A8), IC58.1 (A8), IC59.1 (A8), IC60.1 (A8), IC61.1 (A8), IC62.1 (A8), IC63.1 (A8), IC64.1 (A8), IC65.1 (A8), IC72.1 (A8), IC73.1 (A8), IC74.1 (A8), IC75.1 (A8), IC76.1 (A8), IC77.1 (A8), IC78.1 (A8), IC79.1 (A8), IC80.1 (A8), IC89.1 (A8), IC90.1 (A8), IC91.1 (A8), IC92.1 (A8), IC93.1 (A8), IC94.1 (A8), IC95.1 (A8), IC96.1 (A8), IC97.1 (A8)
- new net MD0: IC44.14 (Q), IC44.2 (D), IC58.14 (Q), IC58.2 (D), IC73.14 (Q), IC73.2 (D), IC90.14 (Q), IC90.2 (D)
- new net MD1: IC45.14 (Q), IC45.2 (D), IC59.14 (Q), IC59.2 (D), IC74.14 (Q), IC74.2 (D), IC91.14 (Q), IC91.2 (D)
- new net MD2: IC46.14 (Q), IC46.2 (D), IC60.14 (Q), IC60.2 (D), IC75.14 (Q), IC75.2 (D), IC92.14 (Q), IC92.2 (D)
- new net MD3: IC47.14 (Q), IC47.2 (D), IC61.14 (Q), IC61.2 (D), IC76.14 (Q), IC76.2 (D), IC93.14 (Q), IC93.2 (D)
- new net MD4: IC48.14 (Q), IC48.2 (D), IC62.14 (Q), IC62.2 (D), IC77.14 (Q), IC77.2 (D), IC94.14 (Q), IC94.2 (D)
- new net MD5: IC49.14 (Q), IC49.2 (D), IC63.14 (Q), IC63.2 (D), IC78.14 (Q), IC78.2 (D), IC95.14 (Q), IC95.2 (D)
- new net MD6: IC50.14 (Q), IC50.2 (D), IC64.14 (Q), IC64.2 (D), IC79.14 (Q), IC79.2 (D), IC96.14 (Q), IC96.2 (D)
- new net MD7: IC51.14 (Q), IC51.2 (D), IC65.14 (Q), IC65.2 (D), IC80.14 (Q), IC80.2 (D), IC97.14 (Q), IC97.2 (D)
- new net MDP_IN: IC43.2 (D), IC57.2 (D), IC72.2 (D), IC89.2 (D)
- new net MDP_OUT: IC43.14 (Q), IC57.14 (Q), IC72.14 (Q), IC89.14 (Q)
- new net ~CAS0~: IC43.15 (~CAS), IC44.15 (~CAS), IC45.15 (~CAS), IC46.15 (~CAS), IC47.15 (~CAS), IC48.15 (~CAS), IC49.15 (~CAS), IC50.15 (~CAS), IC51.15 (~CAS)
- new net ~CAS1~: IC57.15 (~CAS), IC58.15 (~CAS), IC59.15 (~CAS), IC60.15 (~CAS), IC61.15 (~CAS), IC62.15 (~CAS), IC63.15 (~CAS), IC64.15 (~CAS), IC65.15 (~CAS)
- new net ~CAS2~: IC72.15 (~CAS), IC73.15 (~CAS), IC74.15 (~CAS), IC75.15 (~CAS), IC76.15 (~CAS), IC77.15 (~CAS), IC78.15 (~CAS), IC79.15 (~CAS), IC80.15 (~CAS)
- new net ~CAS3~: IC89.15 (~CAS), IC90.15 (~CAS), IC91.15 (~CAS), IC92.15 (~CAS), IC93.15 (~CAS), IC94.15 (~CAS), IC95.15 (~CAS), IC96.15 (~CAS), IC97.15 (~CAS)
- new net ~MWE~: IC43.3 (~W), IC44.3 (~W), IC45.3 (~W), IC46.3 (~W), IC47.3 (~W), IC48.3 (~W), IC49.3 (~W), IC50.3 (~W), IC51.3 (~W), IC57.3 (~W), IC58.3 (~W), IC59.3 (~W), IC60.3 (~W), IC61.3 (~W), IC62.3 (~W), IC63.3 (~W), IC64.3 (~W), IC65.3 (~W), IC72.3 (~W), IC73.3 (~W), IC74.3 (~W), IC75.3 (~W), IC76.3 (~W), IC77.3 (~W), IC78.3 (~W), IC79.3 (~W), IC80.3 (~W), IC89.3 (~W), IC90.3 (~W), IC91.3 (~W), IC92.3 (~W), IC93.3 (~W), IC94.3 (~W), IC95.3 (~W), IC96.3 (~W), IC97.3 (~W)
- new net ~RAS0~: IC43.4 (~RAS), IC44.4 (~RAS), IC45.4 (~RAS), IC46.4 (~RAS), IC47.4 (~RAS), IC48.4 (~RAS), IC49.4 (~RAS), IC50.4 (~RAS), IC51.4 (~RAS)
- new net ~RAS1~: IC57.4 (~RAS), IC58.4 (~RAS), IC59.4 (~RAS), IC60.4 (~RAS), IC61.4 (~RAS), IC62.4 (~RAS), IC63.4 (~RAS), IC64.4 (~RAS), IC65.4 (~RAS)
- new net ~RAS2~: IC72.4 (~RAS), IC73.4 (~RAS), IC74.4 (~RAS), IC75.4 (~RAS), IC76.4 (~RAS), IC77.4 (~RAS), IC78.4 (~RAS), IC79.4 (~RAS), IC80.4 (~RAS)
- new net ~RAS3~: IC89.4 (~RAS), IC90.4 (~RAS), IC91.4 (~RAS), IC92.4 (~RAS), IC93.4 (~RAS), IC94.4 (~RAS), IC95.4 (~RAS), IC96.4 (~RAS), IC97.4 (~RAS)
Other:
- note added: "Bank 0"
- note added: "Bank 1"
- note added: "Bank 2"
- note added: "Bank 3"
